File: OpenC16RamExpansion.kicad_pcb (KiCad board)
At the start: 2 copper layers, 50 x 48.3 mm, 4 parts, among them U1 74LS257, U2 74LS257, U3 4464, U4 4464

Commit message: Working on PCB
Parts:
- added J1: C16-Exp-Port, C16_Cart_Conn:C16_Cart_Conn, F.Cu at (149.5, 142.2)
Connections:
- net Net-(U1-Pad1) renamed /sel
- net Net-(U3-Pad16) renamed //cas
- net Net-(U3-Pad4) renamed /r/w
- net Net-(U3-Pad5) renamed //ras
Routing:
- net //ras: track 13.6 -> 99.0 mm, vias 0 -> 1
- net VCC: track 28.5 -> 95.3 mm
- net /c16_a8: track 0.00 -> 46.1 mm, vias 0 -> 2
- net /c16_a10: track 0.00 -> 43.5 mm, vias 0 -> 1
- net /c16_a14: track 0.00 -> 42.3 mm, vias 0 -> 1
- net /c16_a15: track 0.00 -> 39.7 mm, vias 0 -> 1
- net /c16_a11: track 0.00 -> 38.7 mm, vias 0 -> 1
- net /c16_a9: track 0.00 -> 33.6 mm, vias 0 -> 1
- net /c16_a13: track 0.00 -> 29.3 mm, vias 0 -> 2
- net /c16_a12: track 0.00 -> 25.9 mm, vias 0 -> 1
- net GND: track 34.0 -> 50.6 mm

Commit message: Almost there...
Parts:
- added G***: LOGO, w_logo:Logo_copper_OSHW_6x6mm, B.Cu at (169.4, 127.3)
Routing:
- net /a7: track 0.00 -> 89.3 mm
- net GND: track 50.6 -> 133.5 mm, vias 0 -> 11
- net /a1: track 13.4 -> 95.2 mm
- net /a2: track 13.4 -> 89.3 mm, vias 0 -> 1
- net /a0: track 13.4 -> 84.1 mm, vias 0 -> 2
- net /a3: track 13.4 -> 83.3 mm
- net /c16_a0: track 0.00 -> 68.7 mm, vias 0 -> 2
- net /c16_a1: track 0.00 -> 59.8 mm, vias 0 -> 2
- net /c16_a3: track 0.00 -> 56.2 mm, vias 0 -> 1
- net /c16_a4: track 0.00 -> 50.3 mm, vias 0 -> 1
- net /r/w: track 13.4 -> 61.8 mm, vias 0 -> 2
- net /c16_a2: track 0.00 -> 46.7 mm, vias 0 -> 1
- net /d3: track 0.00 -> 46.6 mm, vias 0 -> 1
- net /sel: track 13.7 -> 57.2 mm, vias 0 -> 1
- net //cas: track 13.4 -> 56.3 mm, vias 0 -> 1
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Other:
- board size 50 x 48.3 mm -> 51.1 x 45 mm
- net class Default: clearance 0.254 -> 0.2032; via_dia 0.8 -> 0.7
- net class Power: clearance 0.254 -> 0.2032; trace_width 0.508 -> 0.4064; via_dia 1.4 -> 1.2
- rule trace_clearance: 0.254 -> 0.2032
- board text added: "V1.0"
- board text added: "https://github.com/SukkoPera/OpenC16RamExpansion"
