File: OpenC16RamExpansion.kicad_pcb (KiCad board)
At the start: 2 copper layers, 52 x 45 mm, 10 parts, among them J1 C16-Exp-Port, U1 74LS257, U2 74LS257, U3 4464, U4 4464

Commit message: Zero pad clearance
Other:
- rule pad_to_mask_clearance: 0.2 -> 0
Changed lines of the file:
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@@
     (pad_size 51 8)
     (pad_drill 0)
-    (pad_to_mask_clearance 0.2)
+    (pad_to_mask_clearance 0)
     (aux_axis_origin 0 0)
     (grid_origin 123.55 142.15)
